File: Digisynth_PCB/Digisynth.kicad_pcb (KiCad board)
At the start: 2 copper layers, 100 x 50 mm, 44 parts, among them J1 Conn_02x02_Counter_Clockwise, J10 Conn_02x04_Counter_Clockwise, J11 Conn_02x02_Counter_Clockwise, J12 AudioJack3_Ground, J13 Conn_01x01_Female, J14 Conn_01x01_Female, J15 Conn_01x03, J16 Conn_01x03, J2 Conn_01x03_Female, J3 Conn_02x03_Counter_Clockwise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

Commit message: Add gerbers
Other:
- board text added: "Potentiometer"
- board text removed: "Potentiometer B"
Changed lines of the file:
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@@
     (visible_elements 7FFFF7FF)
     (pcbplotparams
-      (layerselection 0x010fc_ffffffff)
+      (layerselection 0x010f0_ffffffff)
       (usegerberextensions false)
       (usegerberattributes false)
@@
       (outputformat 1)
       (mirror false)
-      (drillshape 1)
+      (drillshape 0)
       (scaleselection 1)
-      (outputdirectory ""))
+      (outputdirectory "Gerbers/"))
   )
   (net 0 "")
@@
     (effects (font (size 1.5 1.5) (thickness 0.3)))
   )
-  (gr_text "Potentiometer B" (at 91.4 23.5 90) (layer F.SilkS)
+  (gr_text Potentiometer (at 91.4 23.5 90) (layer F.SilkS)
     (effects (font (size 1 1) (thickness 0.2)))
   )
